File: BinBreakout_2/BinBreakout_2.kicad_pcb (KiCad board)
At the start: 2 copper layers, 55 x 19 mm, 7 parts

Commit message: version 1 of the boards. getting printed PCBs from OSH park
Changed lines of the file:
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@@
     (links 6)
     (no_connects 0)
-    (area 100.924999 75.1246 156.075001 97.5274)
+    (area 100.924999 75.924999 156.075001 95.075001)
     (thickness 1.6002)
     (drawings 8)
@@
   )
   (setup
-    (last_trace_width 0.1524)
+    (last_trace_width 0.508)
     (user_trace_width 0.1524)
     (user_trace_width 0.254)
@@
     (user_via 0.6858 0.3302)
     (user_via 0.6858 0.4)
+    (user_via 0.762 0.4572)
     (user_via 1.905 0.3302)
     (uvia_size 0.762)
@@
   (gr_line (start 156 76) (end 156 95) (angle 90) (layer Edge.Cuts) (width 0.15))
   (gr_line (start 156 95) (end 101 95) (angle 90) (layer Edge.Cuts) (width 0.15))
-  (segment (start 111.5 80.8) (end 111.5 81.5) (width 0.254) (layer Bottom) (net 1))
-  (segment (start 111.5 81.5) (end 114.3 84.3) (width 0.254) (layer Bottom) (net 1))
-  (segment (start 114.3 84.3) (end 130.2 84.3) (width 0.254) (layer Bottom) (net 1))
-  (via (at 130.2 84.3) (size 0.6858) (drill 0.3302) (layers Top Bottom) (net 1))
-  (segment (start 130.2 84.3) (end 130.2 81.4) (width 0.254) (layer Top) (net 1))
-  (segment (start 130.2 81.4) (end 130.8 80.8) (width 0.254) (layer Top) (net 1))
-  (segment (start 130.8 80.8) (end 137.3 80.8) (width 0.254) (layer Top) (net 1))
-  (segment (start 112.77 78.26) (end 112.86 78.26) (width 0.254) (layer Bottom) (net 2))
-  (segment (start 112.86 78.26) (end 114.1 79.5) (width 0.254) (layer Bottom) (net 2))
-  (segment (start 114.1 79.5) (end 137.33 79.5) (width 0.254) (layer Bottom) (net 2))
-  (segment (start 137.33 79.5) (end 138.57 78.26) (width 0.254) (layer Bottom) (net 2))
-  (segment (start 114.04 80.8) (end 114.04 81.14) (width 0.254) (layer Bottom) (net 3))
-  (segment (start 114.04 81.14) (end 116.2 83.3) (width 0.254) (layer Bottom) (net 3))
-  (segment (start 116.2 83.3) (end 138.7 83.3) (width 0.254) (layer Bottom) (net 3))
-  (segment (start 138.7 83.3) (end 139.84 82.16) (width 0.254) (layer Bottom) (net 3))
-  (segment (start 139.84 82.16) (end 139.84 80.8) (width 0.254) (layer Bottom) (net 3))
-  (segment (start 115.31 78.26) (end 115.31 78.09) (width 0.254) (layer Top) (net 4))
-  (segment (start 115.31 78.09) (end 116.4 77) (width 0.254) (layer Top) (net 4))
-  (segment (start 139.85 77) (end 141.11 78.26) (width 0.254) (layer Top) (net 4))
-  (segment (start 116.4 77) (end 139.85 77) (width 0.254) (layer Top) (net 4))
-  (segment (start 115.31 78.26) (end 115.44 78.26) (width 0.254) (layer Top) (net 4))
-  (segment (start 116.58 80.8) (end 116.58 81.28) (width 0.254) (layer Bottom) (net 5))
-  (segment (start 116.58 80.8) (end 116.58 80.98) (width 0.381) (layer Top) (net 5))
-  (segment (start 116.58 80.98) (end 119.3 83.7) (width 0.381) (layer Top) (net 5))
-  (segment (start 127 86.4) (end 127 90.5) (width 0.381) (layer Top) (net 5))
-  (segment (start 124.3 83.7) (end 127 86.4) (width 0.381) (layer Top) (net 5))
-  (segment (start 119.3 83.7) (end 124.3 83.7) (width 0.381) (layer Top) (net 5))
-  (segment (start 117.85 78.26) (end 117.86 78.26) (width 0.381) (layer Top) (net 6))
-  (segment (start 117.86 78.26) (end 119.1 79.5) (width 0.381) (layer Top) (net 6))
-  (segment (start 119.1 79.5) (end 123.6 79.5) (width 0.381) (layer Top) (net 6))
-  (segment (start 123.6 79.5) (end 130.5 86.4) (width 0.381) (layer Top) (net 6))
-  (segment (start 130.5 86.4) (end 130.5 90.5) (width 0.381) (layer Top) (net 6))
-  (segment (start 117.85 78.16) (end 117.85 77.85) (width 0.254) (layer Top) (net 6))
+  (segment (start 111.5 80.8) (end 111.5 81.5) (width 0.508) (layer Bottom) (net 1) (status 30))
+  (segment (start 111.5 81.5) (end 114.3 84.3) (width 0.508) (layer Bottom) (net 1) (status 10))
+  (segment (start 114.3 84.3) (end 130.2 84.3) (width 0.508) (layer Bottom) (net 1))
+  (via (at 130.2 84.3) (size 0.762) (drill 0.4572) (layers Top Bottom) (net 1))
+  (segment (start 130.2 84.3) (end 130.2 81.4) (width 0.508) (layer Top) (net 1))
+  (segment (start 130.2 81.4) (end 130.8 80.8) (width 0.508) (layer Top) (net 1))
+  (segment (start 130.8 80.8) (end 137.3 80.8) (width 0.508) (layer Top) (net 1) (status 20))
+  (segment (start 112.77 78.26) (end 112.86 78.26) (width 0.508) (layer Bottom) (net 2) (status 30))
+  (segment (start 112.86 78.26) (end 114.1 79.5) (width 0.508) (layer Bottom) (net 2) (status 10))
+  (segment (start 114.1 79.5) (end 137.33 79.5) (width 0.508) (layer Bottom) (net 2))
+  (segment (start 137.33 79.5) (end 138.57 78.26) (width 0.508) (layer Bottom) (net 2) (status 20))
+  (segment (start 114.04 80.8) (end 114.04 81.14) (width 0.508) (layer Bottom) (net 3) (status 30))
+  (segment (start 114.04 81.14) (end 116.2 83.3) (width 0.508) (layer Bottom) (net 3) (status 10))
+  (segment (start 116.2 83.3) (end 138.7 83.3) (width 0.508) (layer Bottom) (net 3))
+  (segment (start 138.7 83.3) (end 139.84 82.16) (width 0.508) (layer Bottom) (net 3))
+  (segment (start 139.84 82.16) (end 139.84 80.8) (width 0.508) (layer Bottom) (net 3) (status 20))
+  (segment (start 115.31 78.26) (end 115.31 78.09) (width 0.508) (layer Top) (net 4) (status 30))
+  (segment (start 115.31 78.09) (end 116.4 77) (width 0.508) (layer Top) (net 4) (status 10))
+  (segment (start 139.85 77) (end 141.11 78.26) (width 0.508) (layer Top) (net 4) (status 20))
+  (segment (start 116.4 77) (end 139.85 77) (width 0.508) (layer Top) (net 4))
+  (segment (start 115.31 78.26) (end 115.44 78.26) (width 0.508) (layer Top) (net 4) (status 30))
+  (segment (start 116.58 80.8) (end 116.58 81.28) (width 0.508) (layer Bottom) (net 5) (status 30))
+  (segment (start 116.58 80.8) (end 116.58 80.98) (width 0.508) (layer Top) (net 5) (status 30))
+  (segment (start 116.58 80.98) (end 119.3 83.7) (width 0.508) (layer Top) (net 5) (status 10))
+  (segment (start 127 86.4) (end 127 90.5) (width 0.508) (layer Top) (net 5) (status 20))
+  (segment (start 124.3 83.7) (end 127 86.4) (width 0.508) (layer Top) (net 5))
+  (segment (start 119.3 83.7) (end 124.3 83.7) (width 0.508) (layer Top) (net 5))
+  (segment (start 117.85 78.26) (end 117.86 78.26) (width 0.508) (layer Top) (net 6) (status 30))
+  (segment (start 117.86 78.26) (end 119.1 79.5) (width 0.508) (layer Top) (net 6) (status 10))
+  (segment (start 119.1 79.5) (end 123.6 79.5) (width 0.508) (layer Top) (net 6))
+  (segment (start 123.6 79.5) (end 130.5 86.4) (width 0.508) (layer Top) (net 6))
+  (segment (start 130.5 86.4) (end 130.5 90.5) (width 0.508) (layer Top) (net 6) (status 20))
+  (segment (start 117.85 78.16) (end 117.85 77.85) (width 0.508) (layer Top) (net 6) (status 30))
 )
