File: BinBreakout_3/BinBreakout_3.kicad_pcb (KiCad board)
At the start: 2 copper layers, 55 x 19 mm, 7 parts

Commit message: version 1 of the boards. getting printed PCBs from OSH park
Changed lines of the file:
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@@
   )
   (setup
-    (last_trace_width 0.1524)
+    (last_trace_width 0.508)
     (user_trace_width 0.1524)
     (user_trace_width 0.254)
@@
     (user_via 0.6858 0.3302)
     (user_via 0.6858 0.4)
+    (user_via 0.762 0.4572)
     (user_via 1.905 0.3302)
     (uvia_size 0.762)
@@
   (gr_line (start 156 76) (end 156 95) (angle 90) (layer Edge.Cuts) (width 0.15))
   (gr_line (start 156 95) (end 101 95) (angle 90) (layer Edge.Cuts) (width 0.15))
-  (segment (start 111.5 80.8) (end 111.5 81.6) (width 0.254) (layer Bottom) (net 1))
-  (segment (start 135.5 82.6) (end 137.3 80.8) (width 0.254) (layer Bottom) (net 1))
-  (segment (start 112.5 82.6) (end 135.5 82.6) (width 0.254) (layer Bottom) (net 1))
-  (segment (start 111.5 81.6) (end 112.5 82.6) (width 0.254) (layer Bottom) (net 1))
-  (segment (start 111.5 80.8) (end 111.5 81.5) (width 0.254) (layer Bottom) (net 1))
-  (segment (start 112.77 78.26) (end 112.77 78.23) (width 0.254) (layer Bottom) (net 2))
-  (segment (start 112.77 78.23) (end 113.9 77.1) (width 0.254) (layer Bottom) (net 2))
-  (segment (start 137.41 77.1) (end 138.57 78.26) (width 0.254) (layer Bottom) (net 2))
-  (segment (start 113.9 77.1) (end 137.41 77.1) (width 0.254) (layer Bottom) (net 2))
-  (segment (start 112.77 78.26) (end 112.86 78.26) (width 0.254) (layer Bottom) (net 2))
-  (segment (start 114.04 80.8) (end 114.04 81.14) (width 0.254) (layer Bottom) (net 3))
-  (segment (start 114.04 80.8) (end 114.04 83.44) (width 0.381) (layer Top) (net 3))
-  (segment (start 127 85.8) (end 127 90.5) (width 0.381) (layer Top) (net 3))
-  (segment (start 125.8 84.6) (end 127 85.8) (width 0.381) (layer Top) (net 3))
-  (segment (start 115.2 84.6) (end 125.8 84.6) (width 0.381) (layer Top) (net 3))
-  (segment (start 114.04 83.44) (end 115.2 84.6) (width 0.381) (layer Top) (net 3))
-  (segment (start 115.31 78.26) (end 115.31 82.79) (width 0.381) (layer Top) (net 4))
-  (segment (start 130.5 85.6) (end 130.5 90.5) (width 0.381) (layer Top) (net 4))
-  (segment (start 128.6 83.7) (end 130.5 85.6) (width 0.381) (layer Top) (net 4))
-  (segment (start 116.22 83.7) (end 128.6 83.7) (width 0.381) (layer Top) (net 4))
-  (segment (start 115.31 82.79) (end 116.22 83.7) (width 0.381) (layer Top) (net 4))
-  (segment (start 115.31 78.26) (end 115.31 78.09) (width 0.254) (layer Top) (net 4))
-  (segment (start 115.31 78.26) (end 115.44 78.26) (width 0.254) (layer Top) (net 4))
+  (segment (start 111.5 80.8) (end 111.5 81.6) (width 0.508) (layer Bottom) (net 1))
+  (segment (start 135.5 82.6) (end 137.3 80.8) (width 0.508) (layer Bottom) (net 1))
+  (segment (start 112.5 82.6) (end 135.5 82.6) (width 0.508) (layer Bottom) (net 1))
+  (segment (start 111.5 81.6) (end 112.5 82.6) (width 0.508) (layer Bottom) (net 1))
+  (segment (start 111.5 80.8) (end 111.5 81.5) (width 0.508) (layer Bottom) (net 1))
+  (segment (start 112.77 78.26) (end 112.77 78.23) (width 0.508) (layer Bottom) (net 2))
+  (segment (start 112.77 78.23) (end 113.9 77.1) (width 0.508) (layer Bottom) (net 2))
+  (segment (start 137.41 77.1) (end 138.57 78.26) (width 0.508) (layer Bottom) (net 2))
+  (segment (start 113.9 77.1) (end 137.41 77.1) (width 0.508) (layer Bottom) (net 2))
+  (segment (start 112.77 78.26) (end 112.86 78.26) (width 0.508) (layer Bottom) (net 2))
+  (segment (start 114.04 80.8) (end 114.04 81.14) (width 0.508) (layer Bottom) (net 3))
+  (segment (start 114.04 80.8) (end 114.04 83.44) (width 0.508) (layer Top) (net 3))
+  (segment (start 127 85.8) (end 127 90.5) (width 0.508) (layer Top) (net 3))
+  (segment (start 125.8 84.6) (end 127 85.8) (width 0.508) (layer Top) (net 3))
+  (segment (start 115.2 84.6) (end 125.8 84.6) (width 0.508) (layer Top) (net 3))
+  (segment (start 114.04 83.44) (end 115.2 84.6) (width 0.508) (layer Top) (net 3))
+  (segment (start 115.31 78.26) (end 115.31 82.79) (width 0.508) (layer Top) (net 4))
+  (segment (start 130.5 85.6) (end 130.5 90.5) (width 0.508) (layer Top) (net 4))
+  (segment (start 128.6 83.7) (end 130.5 85.6) (width 0.508) (layer Top) (net 4))
+  (segment (start 116.22 83.7) (end 128.6 83.7) (width 0.508) (layer Top) (net 4))
+  (segment (start 115.31 82.79) (end 116.22 83.7) (width 0.508) (layer Top) (net 4))
+  (segment (start 115.31 78.26) (end 115.31 78.09) (width 0.508) (layer Top) (net 4))
+  (segment (start 115.31 78.26) (end 115.44 78.26) (width 0.508) (layer Top) (net 4))
   (segment (start 116.58 80.8) (end 116.58 81.28) (width 0.254) (layer Bottom) (net 11))
   (segment (start 117.85 78.26) (end 117.86 78.26) (width 0.381) (layer Top) (net 12))
