File: FarmMonitor/FarmMonitor.kicad_pcb (KiCad board)
At the start: 2 copper layers, 65 x 55 mm, 24 parts

Commit message: version 1 of the boards. getting printed PCBs from OSH park
Parts:
- removed npn1: Q_NPN_EBC, TO_SOT_Packages_THT:TO-92_Inline_Narrow_Oval
- added C1: 0.1uF, Capacitors_SMD:C_0805_HandSoldering, B.Cu at (106.5, 119.7)
- added C2: 0.1 uF, Capacitors_SMD:C_0805_HandSoldering, B.Cu at (92.3, 121.9)
- added LED4: LED, LEDs:LED_D5.0mm, F.Cu at (105.2, 100.0)
- added PNP1: Q_PNP_EBC, TO_SOT_Packages_THT:TO-92_Inline_Narrow_Oval, F.Cu at (105.8, 109.7)
- added R5: 200, Resistors_SMD:R_0805_HandSoldering, B.Cu at (112.1, 99.3)
- added R6: 1K, Resistors_SMD:R_0805_HandSoldering, B.Cu at (108.1, 104.1)
- R2, R3: value 120 -> 200; moved to B.Cu
- R4: value 120 -> 200
- temperature_1: footprint TO_SOT_Packages_THT:TO-92_Horizontal2_Inline_Narrow_Oval -> TO_SOT_Packages_THT:TO-92_Inline_Narrow_Oval
- moved R3 21.7 mm to (87.2, 104.2)
- moved temperature_1 11.3 mm to (77.9, 123.7), turned to 0 degrees
- moved R2 11.2 mm to (97.7, 104.2)
- moved LED2 10.6 mm to (84.8, 100.0)
- moved LED1 9.21 mm to (94.6, 100.0)
- moved LED3 5.10 mm to (70.0, 113.9)
- moved R4 4.21 mm to (68.7, 120.3)
- moved button_1 2.09 mm to (77.1, 108.0)
- moved button_2 0.92 mm to (93.0, 108.0)
- moved temperature_2 0.30 mm to (68.5, 130.1)
Connections:
- rpi_header_1 pad 29: /restart -> /start_inhibit
- rpi_header_1 pad 31: Net-(rpi_header_1-Pad31) -> /led_4
Routing:
- net GND: track 202.1 -> 254.7 mm, vias 3 -> 4
- net /start_inhibit: track 0.00 -> 19.1 mm, vias 0 -> 1
- net /restart: track 17.6 -> 0.00 mm
- net /led_4: track 0.00 -> 11.4 mm
- net Net-(LED2-Pad1): track 14.7 -> 4.63 mm
- net /feedback_led: track 14.5 -> 7.47 mm
- net Net-(LED4-Pad1): track 0.00 -> 5.84 mm
- net /SDA: track 51.7 -> 55.4 mm
- net Net-(R1-Pad2): track 56.7 -> 53.4 mm
- net /button: track 24.1 -> 21.9 mm
- net /status_led: track 8.62 -> 6.71 mm
- net +5V: track 111.5 -> 113.3 mm, vias 2 -> 4
- net Net-(LED3-Pad1): track 7.36 -> 6.42 mm
- net /SCL: track 62.9 -> 62.3 mm
